File: Schematics/Kicad 5/Arduino_Uno_R3.sch (KiCad schematic (older format))
At the start: 65 parts

Commit message: addded Arduino_Uno_Header symbol
Parts:
- removed P? (x4): CONN_01X01, Socket_Arduino_Uno:Arduino_1pin, symbol Connector_Generic:Conn_01x01
- P? (x2): footprint Socket_Arduino_Uno:Socket_Strip_Arduino_1x08 -> ~; symbol Connector_Generic:Conn_01x08 -> Arduino_Uno_R3:CONN_01X08
- P?: footprint Socket_Arduino_Uno:Socket_Strip_Arduino_1x10 -> ~; symbol Connector_Generic:Conn_01x10 -> Arduino_Uno_R3:CONN_01X10
- P?: footprint Socket_Arduino_Uno:Socket_Strip_Arduino_1x06 -> ~; symbol Connector_Generic:Conn_01x06 -> Arduino_Uno_R3:CONN_01X06
Connections:
- no-connect marks 15 -> 11
Other:
- note removed: "Holes"
